File: KiCAD_Files/OpenDTU_Breakout.kicad_pcb (KiCad board)
At the start: 2 copper layers, 35 x 55 mm, 12 parts, among them J1 I2C, J2 Power, J3 Conn_01x03_Male, U1 ESP32-DEVKITC-32D, U2 NRF24L01_Breakout

Commit message: flipped and rotated J1 and J3
Parts:
- J1, J3: moved to B.Cu
- turned J1 to 90 degrees
- turned J3 to 90 degrees
Other:
- board text added: "REV3"
- board text removed: "REV2"
